File: hardware/MIDI-clock-Eurorack-adapter.kicad_sch (KiCad schematic)
At the start: 26 parts, among them J1 CLOCK, J2 RUN, J3 Conn_02x05_Odd_Even, Q1 2N3904, U1 TL072

Commit message: Update schematic
Parts:
- removed C3: 100n, symbol Device:C_Small
- removed C4, C5: 10u, symbol Device:C_Polarized_US
- removed D1, D2: 1N5819, Diode_THT:D_DO-41_SOD81_P10.16mm_Horizontal, symbol Diode:1N5819
- removed D3, D4: 1N4148, Diode_THT:D_DO-35_SOD27_P7.62mm_Horizontal, symbol Diode:1N4148
- removed J3: Conn_02x05_Odd_Even, symbol Connector_Generic:Conn_02x05_Odd_Even
- removed R10, R4: 15K, symbol Device:R_US
- removed R2: 33K, symbol Device:R_US
- removed R8: 100K, symbol Device:R_US
Connections:
- net +12V: no longer C2.2, D5.2 (A), R1.1, U1.8 (V+)
- net CLOCK: now also R5.1, U1.6 (-)
- net GND: now also C2.1, R1.2, U1.4 (V-)
- net RUN: now also U1.1, U1.2 (-)
- net at A1.5 (D2): now also R1.1, U1.5 (+); no longer U1.6 (-)
- net at A1.6 (D3), R9.1: now also U1.3 (+); no longer U1.2 (-)
- net +5V: now reaches A1.27 (+5V)
- net +5V: now also C2.2, D5.2 (A), U1.8 (V+)
- removed net Vref: R1.2, U1.3 (+), U1.5 (+)
- no-connect marks 26 -> 25
Other:
- moved on the sheet: C2, D5, J1, J2, Q1, R3, R5, R6, R7, R9, U1B, U1C

Commit message: Update schematic
Parts:
- removed U1: TL072, Package_DIP:DIP-8_W7.62mm_Socket_LongPads, symbol Amplifier_Operational:TL072
- added U1: MCP6002-xP, Package_DIP:DIP-8_W7.62mm_Socket_LongPads, symbol Amplifier_Operational:MCP6002-xP
Connections:
- net +5V: now also U1.8 (V+)
- net CLOCK: now also U1.1, U1.2 (-)
- net GND: now also U1.4 (V-)
- net RUN: now also U1.6 (-), U1.7
- net at R1.1: now also A1.6 (D3), U1.3 (+); no longer A1.5 (D2)
- net at R9.1: now also A1.12 (D9), U1.5 (+); no longer A1.6 (D3)
- no-connect marks 25 -> 26
Other:
- moved on the sheet: J1, R1, R5
